Commit message: feat: add headless mode and configurable spawn poses to simulation and SLAM launch files

File: src/mir_description/urdf/mir.urdf.xacro (robot description, xacro)
@@ -64,5 +64,5 @@
     <child link="left_wheel_link"/>
     <axis xyz="0 1 0"/>
-    <limit effort="100" velocity="20.0"/>
+    <limit effort="10000" velocity="20.0"/>
   </joint>
   <link name="left_wheel_link">
@@ -96,5 +96,5 @@
     <child link="right_wheel_link"/>
     <axis xyz="0 1 0"/>
-    <limit effort="100" velocity="20.0"/>
+    <limit effort="10000" velocity="20.0"/>
   </joint>
   <link name="right_wheel_link">
@@ -429,6 +429,6 @@
   </gazebo>
   <gazebo reference="fl_caster_wheel_link">
-    <mu1 value="1"/>
-    <mu2 value="1"/>
+    <mu1 value="0.0"/>
+    <mu2 value="0.0"/>
     <kp value="10000000.0"/>
     <kd value="1.0"/>
@@ -436,6 +436,6 @@
   </gazebo>
   <gazebo reference="fr_caster_wheel_link">
-    <mu1 value="1"/>
-    <mu2 value="1"/>
+    <mu1 value="0.0"/>
+    <mu2 value="0.0"/>
     <kp value="10000000.0"/>
     <kd value="1.0"/>
@@ -443,6 +443,6 @@
   </gazebo>
   <gazebo reference="bl_caster_wheel_link">
-    <mu1 value="1"/>
-    <mu2 value="1"/>
+    <mu1 value="0.0"/>
+    <mu2 value="0.0"/>
     <kp value="10000000.0"/>
     <kd value="1.0"/>
@@ -450,30 +450,11 @@
   </gazebo>
   <gazebo reference="br_caster_wheel_link">
-    <mu1 value="1"/>
-    <mu2 value="1"/>
-    <kp value="10000000.0"/>
-    <kd value="1.0"/>
-    <minDepth>0.01</minDepth>
-  </gazebo>
-  <!-- Gazebo Harmonic: native DiffDrive plugin actuates wheels directly from
-       /cmd_vel and publishes /odom + TF without a separate ROS controller. -->
+    <mu1 value="0.0"/>
+    <mu2 value="0.0"/>
+    <kp value="10000000.0"/>
+    <kd value="1.0"/>
+    <minDepth>0.01</minDepth>
+  </gazebo>
   <gazebo>
-    <plugin filename="gz-sim-diff-drive-system"
-            name="gz::sim::systems::DiffDrive">
-      <!-- wheel joints as they appear in the URDF -->
-      <left_joint>left_wheel_joint</left_joint>
-      <right_joint>right_wheel_joint</right_joint>
-      <!-- physical parameters from the URDF -->
-      <wheel_separation>0.445208</wheel_separation>
-      <wheel_radius>0.0625</wheel_radius>
-      <!-- topics — bridged via ros_gz_bridge in spawn_maze.launch.py -->
-      <topic>cmd_vel</topic>
-      <odom_topic>odom</odom_topic>
-      <!-- /tf is what ros_gz_bridge watches; /gazebo/tf was never bridged -->
-      <tf_topic>gazebo_tf</tf_topic>
-      <frame_id>odom</frame_id>
-      <child_frame_id>base_footprint</child_frame_id>
-      <odom_publish_frequency>50</odom_publish_frequency>
-    </plugin>
     <!-- Gazebo Harmonic: Joint State Publisher to publish wheel/caster angles -->
     <plugin filename="gz-sim-joint-state-publisher-system"

File: src/mobile_manipulator_description/urdf/mobile_manipulator.gazebo.xacro (robot description, xacro)
@@ -3,5 +3,5 @@
   <!-- Include the base URDF/Xacro -->
   <xacro:include filename="$(find mobile_manipulator_description)/urdf/mobile_manipulator.urdf.xacro" />
-  <!-- Gazebo-specific joint state publisher for the UR5e joints -->
+  <!-- Gazebo-specific joint state publisher for the UR5e joints and passive caster joints -->
   <gazebo>
     <plugin filename="gz-sim-joint-state-publisher-system"
@@ -14,4 +14,12 @@
       <joint_name>ur5e_wrist_2_joint</joint_name>
       <joint_name>ur5e_wrist_3_joint</joint_name>
+      <joint_name>fl_caster_rotation_joint</joint_name>
+      <joint_name>fl_caster_wheel_joint</joint_name>
+      <joint_name>fr_caster_rotation_joint</joint_name>
+      <joint_name>fr_caster_wheel_joint</joint_name>
+      <joint_name>bl_caster_rotation_joint</joint_name>
+      <joint_name>bl_caster_wheel_joint</joint_name>
+      <joint_name>br_caster_rotation_joint</joint_name>
+      <joint_name>br_caster_wheel_joint</joint_name>
     </plugin>
   </gazebo>
@@ -70,4 +78,37 @@
       <state_interface name="velocity" />
     </joint>
+    <!-- Passive Caster Joints -->
+    <joint name="fl_caster_rotation_joint">
+      <state_interface name="position" />
+      <state_interface name="velocity" />
+    </joint>
+    <joint name="fl_caster_wheel_joint">
+      <state_interface name="position" />
+      <state_interface name="velocity" />
+    </joint>
+    <joint name="fr_caster_rotation_joint">
+      <state_interface name="position" />
+      <state_interface name="velocity" />
+    </joint>
+    <joint name="fr_caster_wheel_joint">
+      <state_interface name="position" />
+      <state_interface name="velocity" />
+    </joint>
+    <joint name="bl_caster_rotation_joint">
+      <state_interface name="position" />
+      <state_interface name="velocity" />
+    </joint>
+    <joint name="bl_caster_wheel_joint">
+      <state_interface name="position" />
+      <state_interface name="velocity" />
+    </joint>
+    <joint name="br_caster_rotation_joint">
+      <state_interface name="position" />
+      <state_interface name="velocity" />
+    </joint>
+    <joint name="br_caster_wheel_joint">
+      <state_interface name="position" />
+      <state_interface name="velocity" />
+    </joint>
   </ros2_control>
   <!-- Gazebo ros2_control plugin -->

File: src/mobile_manipulator_description/urdf/mobile_manipulator.urdf.xacro (robot description, xacro)
@@ -29,5 +29,5 @@
       <origin xyz="0.0 0.0 -0.15" rpy="0.0 0.0 0.0" />
       <geometry>
-        <cylinder radius="0.50" length="0.40" />
+        <cylinder radius="0.50" length="0.30" />
       </geometry>
     </collision>

Commit message: feat: initialize mobile_manipulator_nav package with custom BT nodes, navigation launch configurations, and simulation environment updates.

File: src/mir_description/urdf/mir.urdf.xacro (robot description, xacro)
@@ -26,10 +26,12 @@
       </material>
     </visual>
-    <collision>
-      <origin rpy="0 0 0" xyz="0.037646 0 0"/>
-      <geometry>
-        <mesh filename="package://mir_description/meshes/collision/mir_100_base.stl"/>
-      </geometry>
-    </collision>
+    <!--
+    <collision>
+      <origin rpy="0 0 0" xyz="0.037646 0 0.18"/>
+      <geometry>
+        <box size="0.95 0.65 0.25"/>
+      </geometry>
+    </collision>
+    -->
   </link>
   <gazebo reference="base_link">
@@ -60,5 +62,5 @@
   <link name="us_2_frame"/>
   <joint name="left_wheel_joint" type="continuous">
-    <origin rpy="0 0 0" xyz="0.0 0.222604 0.0625"/>
+    <origin rpy="0 0 0" xyz="0.0 0.222604 0.061"/>
     <parent link="base_link"/>
     <child link="left_wheel_link"/>
@@ -92,5 +94,5 @@
   </gazebo>
   <joint name="right_wheel_joint" type="continuous">
-    <origin rpy="0 0 0" xyz="0.0 -0.222604 0.0625"/>
+    <origin rpy="0 0 0" xyz="0.0 -0.222604 0.061"/>
     <parent link="base_link"/>
     <child link="right_wheel_link"/>
@@ -124,5 +126,5 @@
   </gazebo>
   <!-- caster hub -->
-  <joint name="fl_caster_rotation_joint" type="continuous">
+  <joint name="fl_caster_rotation_joint" type="fixed">
     <origin rpy="0 0 0" xyz="0.34134600000000004 0.203 0.1565"/>
     <parent link="base_link"/>
@@ -147,10 +149,4 @@
       </material>
     </visual>
-    <collision>
-      <origin rpy="0 0 0" xyz="0 0 0"/>
-      <geometry>
-        <mesh filename="package://mir_description/meshes/collision/caster_wheel_base.stl"/>
-      </geometry>
-    </collision>
   </link>
   <gazebo reference="fl_caster_rotation_link">
@@ -158,5 +154,5 @@
   </gazebo>
   <!-- caster wheel -->
-  <joint name="fl_caster_wheel_joint" type="continuous">
+  <joint name="fl_caster_wheel_joint" type="fixed">
     <origin rpy="0 0 0" xyz="-0.0382 0 -0.094"/>
     <parent link="fl_caster_rotation_link"/>
@@ -190,5 +186,5 @@
   </gazebo>
   <!-- caster hub -->
-  <joint name="fr_caster_rotation_joint" type="continuous">
+  <joint name="fr_caster_rotation_joint" type="fixed">
     <origin rpy="0 0 0" xyz="0.34134600000000004 -0.203 0.1565"/>
     <parent link="base_link"/>
@@ -213,10 +209,4 @@
       </material>
     </visual>
-    <collision>
-      <origin rpy="0 0 0" xyz="0 0 0"/>
-      <geometry>
-        <mesh filename="package://mir_description/meshes/collision/caster_wheel_base.stl"/>
-      </geometry>
-    </collision>
   </link>
   <gazebo reference="fr_caster_rotation_link">
@@ -224,5 +214,5 @@
   </gazebo>
   <!-- caster wheel -->
-  <joint name="fr_caster_wheel_joint" type="continuous">
+  <joint name="fr_caster_wheel_joint" type="fixed">
     <origin rpy="0 0 0" xyz="-0.0382 0 -0.094"/>
     <parent link="fr_caster_rotation_link"/>
@@ -256,5 +246,5 @@
   </gazebo>
   <!-- caster hub -->
-  <joint name="bl_caster_rotation_joint" type="continuous">
+  <joint name="bl_caster_rotation_joint" type="fixed">
     <origin rpy="0 0 0" xyz="-0.270154 0.203 0.1565"/>
     <parent link="base_link"/>
@@ -279,10 +269,4 @@
       </material>
     </visual>
-    <collision>
-      <origin rpy="0 0 0" xyz="0 0 0"/>
-      <geometry>
-        <mesh filename="package://mir_description/meshes/collision/caster_wheel_base.stl"/>
-      </geometry>
-    </collision>
   </link>
   <gazebo reference="bl_caster_rotation_link">
@@ -290,5 +274,5 @@
   </gazebo>
   <!-- caster wheel -->
-  <joint name="bl_caster_wheel_joint" type="continuous">
+  <joint name="bl_caster_wheel_joint" type="fixed">
     <origin rpy="0 0 0" xyz="-0.0382 0 -0.094"/>
     <parent link="bl_caster_rotation_link"/>
@@ -322,5 +306,5 @@
   </gazebo>
   <!-- caster hub -->
-  <joint name="br_caster_rotation_joint" type="continuous">
+  <joint name="br_caster_rotation_joint" type="fixed">
     <origin rpy="0 0 0" xyz="-0.270154 -0.203 0.1565"/>
     <parent link="base_link"/>
@@ -345,10 +329,4 @@
       </material>
     </visual>
-    <collision>
-      <origin rpy="0 0 0" xyz="0 0 0"/>
-      <geometry>
-        <mesh filename="package://mir_description/meshes/collision/caster_wheel_base.stl"/>
-      </geometry>
-    </collision>
   </link>
   <gazebo reference="br_caster_rotation_link">
@@ -356,5 +334,5 @@
   </gazebo>
   <!-- caster wheel -->
-  <joint name="br_caster_wheel_joint" type="continuous">
+  <joint name="br_caster_wheel_joint" type="fixed">
     <origin rpy="0 0 0" xyz="-0.0382 0 -0.094"/>
     <parent link="br_caster_rotation_link"/>
@@ -415,44 +393,44 @@
   </transmission>
   <gazebo reference="left_wheel_link">
-    <mu1 value="200"/>
-    <mu2 value="200"/>
-    <kp value="10000000.0"/>
-    <kd value="1.0"/>
-    <minDepth>0.01</minDepth>
+    <mu1>1.0</mu1>
+    <mu2>1.0</mu2>
+    <kp>10000000.0</kp>
+    <kd>1.0</kd>
+    <minDepth>0.001</minDepth>
   </gazebo>
   <gazebo reference="right_wheel_link">
-    <mu1 value="200"/>
-    <mu2 value="200"/>
-    <kp value="10000000.0"/>
-    <kd value="1.0"/>
-    <minDepth>0.01</minDepth>
+    <mu1>1.0</mu1>
+    <mu2>1.0</mu2>
+    <kp>10000000.0</kp>
+    <kd>1.0</kd>
+    <minDepth>0.001</minDepth>
   </gazebo>
   <gazebo reference="fl_caster_wheel_link">
-    <mu1 value="0.0"/>
-    <mu2 value="0.0"/>
-    <kp value="10000000.0"/>
-    <kd value="1.0"/>
-    <minDepth>0.01</minDepth>
+    <mu1>0.0</mu1>
+    <mu2>0.0</mu2>
+    <kp>10000000.0</kp>
+    <kd>1.0</kd>
+    <minDepth>0.001</minDepth>
   </gazebo>
   <gazebo reference="fr_caster_wheel_link">
-    <mu1 value="0.0"/>
-    <mu2 value="0.0"/>
-    <kp value="10000000.0"/>
-    <kd value="1.0"/>
-    <minDepth>0.01</minDepth>
+    <mu1>0.0</mu1>
+    <mu2>0.0</mu2>
+    <kp>10000000.0</kp>
+    <kd>1.0</kd>
+    <minDepth>0.001</minDepth>
   </gazebo>
   <gazebo reference="bl_caster_wheel_link">
-    <mu1 value="0.0"/>
-    <mu2 value="0.0"/>
-    <kp value="10000000.0"/>
-    <kd value="1.0"/>
-    <minDepth>0.01</minDepth>
+    <mu1>0.0</mu1>
+    <mu2>0.0</mu2>
+    <kp>10000000.0</kp>
+    <kd>1.0</kd>
+    <minDepth>0.001</minDepth>
   </gazebo>
   <gazebo reference="br_caster_wheel_link">
-    <mu1 value="0.0"/>
-    <mu2 value="0.0"/>
-    <kp value="10000000.0"/>
-    <kd value="1.0"/>
-    <minDepth>0.01</minDepth>
+    <mu1>0.0</mu1>
+    <mu2>0.0</mu2>
+    <kp>10000000.0</kp>
+    <kd>1.0</kd>
+    <minDepth>0.001</minDepth>
   </gazebo>
   <gazebo>

File: src/mobile_manipulator_description/urdf/mobile_manipulator.gazebo.xacro (robot description, xacro)
@@ -25,10 +25,10 @@
   </gazebo>
   <!-- Enable self-collision for the arm links in Gazebo -->
-  <gazebo reference="ur5e_shoulder_link"><self_collide>true</self_collide></gazebo>
-  <gazebo reference="ur5e_upper_arm_link"><self_collide>true</self_collide></gazebo>
-  <gazebo reference="ur5e_forearm_link"><self_collide>true</self_collide></gazebo>
-  <gazebo reference="ur5e_wrist_1_link"><self_collide>true</self_collide></gazebo>
-  <gazebo reference="ur5e_wrist_2_link"><self_collide>true</self_collide></gazebo>
-  <gazebo reference="ur5e_wrist_3_link"><self_collide>true</self_collide></gazebo>
+  <gazebo reference="ur5e_shoulder_link"><self_collide>false</self_collide></gazebo>
+  <gazebo reference="ur5e_upper_arm_link"><self_collide>false</self_collide></gazebo>
+  <gazebo reference="ur5e_forearm_link"><self_collide>false</self_collide></gazebo>
+  <gazebo reference="ur5e_wrist_1_link"><self_collide>false</self_collide></gazebo>
+  <gazebo reference="ur5e_wrist_2_link"><self_collide>false</self_collide></gazebo>
+  <gazebo reference="ur5e_wrist_3_link"><self_collide>false</self_collide></gazebo>
   <!-- ros2_control configuration for Gazebo Harmonic -->
   <ros2_control name="gz_ros2_control" type="system">
@@ -86,37 +86,4 @@
       <state_interface name="velocity" />
     </joint>
-    <!-- Passive Caster Joints -->
-    <joint name="fl_caster_rotation_joint">
-      <state_interface name="position" />
-      <state_interface name="velocity" />
-    </joint>
-    <joint name="fl_caster_wheel_joint">
-      <state_interface name="position" />
-      <state_interface name="velocity" />
-    </joint>
-    <joint name="fr_caster_rotation_joint">
-      <state_interface name="position" />
-      <state_interface name="velocity" />
-    </joint>
-    <joint name="fr_caster_wheel_joint">
-      <state_interface name="position" />
-      <state_interface name="velocity" />
-    </joint>
-    <joint name="bl_caster_rotation_joint">
-      <state_interface name="position" />
-      <state_interface name="velocity" />
-    </joint>
-    <joint name="bl_caster_wheel_joint">
-      <state_interface name="position" />
-      <state_interface name="velocity" />
-    </joint>
-    <joint name="br_caster_rotation_joint">
-      <state_interface name="position" />
-      <state_interface name="velocity" />
-    </joint>
-    <joint name="br_caster_wheel_joint">
-      <state_interface name="position" />
-      <state_interface name="velocity" />
-    </joint>
   </ros2_control>
   <!-- Gazebo ros2_control plugin -->

Commit message: feat: replace ros2_control diff_drive_controller with native Gazebo DiffDrive plugin and ros_gz_bridge

File: src/mir_description/urdf/mir.urdf.xacro (robot description, xacro)
@@ -395,42 +395,26 @@
     <mu1>1.0</mu1>
     <mu2>1.0</mu2>
-    <kp>10000000.0</kp>
-    <kd>1.0</kd>
-    <minDepth>0.001</minDepth>
+    <fdir1>1 0 0</fdir1>
   </gazebo>
   <gazebo reference="right_wheel_link">
     <mu1>1.0</mu1>
     <mu2>1.0</mu2>
-    <kp>10000000.0</kp>
-    <kd>1.0</kd>
-    <minDepth>0.001</minDepth>
+    <fdir1>1 0 0</fdir1>
   </gazebo>
   <gazebo reference="fl_caster_wheel_link">
-    <mu1>0.0</mu1>
-    <mu2>0.0</mu2>
-    <kp>10000000.0</kp>
-    <kd>1.0</kd>
-    <minDepth>0.001</minDepth>
+    <mu1>0.001</mu1>
+    <mu2>0.001</mu2>
   </gazebo>
   <gazebo reference="fr_caster_wheel_link">
-    <mu1>0.0</mu1>
-    <mu2>0.0</mu2>
-    <kp>10000000.0</kp>
-    <kd>1.0</kd>
-    <minDepth>0.001</minDepth>
+    <mu1>0.001</mu1>
+    <mu2>0.001</mu2>
   </gazebo>
   <gazebo reference="bl_caster_wheel_link">
-    <mu1>0.0</mu1>
-    <mu2>0.0</mu2>
-    <kp>10000000.0</kp>
-    <kd>1.0</kd>
-    <minDepth>0.001</minDepth>
+    <mu1>0.001</mu1>
+    <mu2>0.001</mu2>
   </gazebo>
   <gazebo reference="br_caster_wheel_link">
-    <mu1>0.0</mu1>
-    <mu2>0.0</mu2>
-    <kp>10000000.0</kp>
-    <kd>1.0</kd>
-    <minDepth>0.001</minDepth>
+    <mu1>0.001</mu1>
+    <mu2>0.001</mu2>
   </gazebo>
   <gazebo>

File: src/mobile_manipulator_description/urdf/mobile_manipulator.gazebo.xacro (robot description, xacro)
@@ -32,19 +32,36 @@
   <gazebo reference="ur5e_wrist_3_link"><self_collide>false</self_collide></gazebo>
   <!-- ros2_control configuration for Gazebo Harmonic -->
+  <!-- Native Gazebo DiffDrive plugin (force/torque based - works with DART physics) -->
+  <gazebo>
+    <plugin filename="gz-sim-diff-drive-system"
+            name="gz::sim::systems::DiffDrive">
+      <left_joint>left_wheel_joint</left_joint>
+      <right_joint>right_wheel_joint</right_joint>
+      <wheel_separation>0.445208</wheel_separation>
+      <wheel_radius>0.0625</wheel_radius>
+      <odom_publish_frequency>50</odom_publish_frequency>
+      <max_linear_acceleration>1.0</max_linear_acceleration>
+      <min_linear_acceleration>-1.0</min_linear_acceleration>
+      <max_angular_acceleration>2.0</max_angular_acceleration>
+      <min_angular_acceleration>-2.0</min_angular_acceleration>
+      <max_linear_velocity>0.5</max_linear_velocity>
+      <min_linear_velocity>-0.5</min_linear_velocity>
+      <max_angular_velocity>1.0</max_angular_velocity>
+      <min_angular_velocity>-1.0</min_angular_velocity>
+      <topic>cmd_vel_gz</topic>
+      <odom_topic>odom_gz</odom_topic>
+      <frame_id>odom</frame_id>
+      <child_frame_id>base_footprint</child_frame_id>
+      <tf_topic>tf_gz</tf_topic>
+      <publish_odom>true</publish_odom>
+      <publish_odom_tf>true</publish_odom_tf>
+      <publish_wheel_tf>false</publish_wheel_tf>
+    </plugin>
+  </gazebo>
+  <!-- ros2_control for UR5e arm only -->
   <ros2_control name="gz_ros2_control" type="system">
     <hardware>
       <plugin>gz_ros2_control/GazeboSimSystem</plugin>
     </hardware>
-    <!-- MiR250 Base Wheels -->
-    <joint name="left_wheel_joint">
-      <command_interface name="velocity" />
-      <state_interface name="position" />
-      <state_interface name="velocity" />
-    </joint>
-    <joint name="right_wheel_joint">
-      <command_interface name="velocity" />
-      <state_interface name="position" />
-      <state_interface name="velocity" />
-    </joint>
     <!-- UR5e Arm Joints -->
     <joint name="ur5e_shoulder_pan_joint">
