Commit message: feat: add navigation bringup launch files and configure collision monitoring for mobile manipulator

File: src/mir_description/urdf/mir.urdf.xacro (robot description, xacro)
@@ -126,5 +126,5 @@
   </gazebo>
   <!-- caster hub -->
-  <joint name="fl_caster_rotation_joint" type="fixed">
+  <joint name="fl_caster_rotation_joint" type="continuous">
     <origin rpy="0 0 0" xyz="0.34134600000000004 0.203 0.1565"/>
     <parent link="base_link"/>
@@ -184,7 +184,9 @@
   <gazebo reference="fl_caster_wheel_link">
     <material>Gazebo/FlatBlack</material>
+    <mu1>0.01</mu1>
+    <mu2>0.01</mu2>
   </gazebo>
   <!-- caster hub -->
-  <joint name="fr_caster_rotation_joint" type="fixed">
+  <joint name="fr_caster_rotation_joint" type="continuous">
     <origin rpy="0 0 0" xyz="0.34134600000000004 -0.203 0.1565"/>
     <parent link="base_link"/>
@@ -244,7 +246,9 @@
   <gazebo reference="fr_caster_wheel_link">
     <material>Gazebo/FlatBlack</material>
+    <mu1>0.01</mu1>
+    <mu2>0.01</mu2>
   </gazebo>
   <!-- caster hub -->
-  <joint name="bl_caster_rotation_joint" type="fixed">
+  <joint name="bl_caster_rotation_joint" type="continuous">
     <origin rpy="0 0 0" xyz="-0.270154 0.203 0.1565"/>
     <parent link="base_link"/>
@@ -304,7 +308,9 @@
   <gazebo reference="bl_caster_wheel_link">
     <material>Gazebo/FlatBlack</material>
+    <mu1>0.01</mu1>
+    <mu2>0.01</mu2>
   </gazebo>
   <!-- caster hub -->
-  <joint name="br_caster_rotation_joint" type="fixed">
+  <joint name="br_caster_rotation_joint" type="continuous">
     <origin rpy="0 0 0" xyz="-0.270154 -0.203 0.1565"/>
     <parent link="base_link"/>
@@ -364,4 +370,6 @@
   <gazebo reference="br_caster_wheel_link">
     <material>Gazebo/FlatBlack</material>
+    <mu1>0.01</mu1>
+    <mu2>0.01</mu2>
   </gazebo>
   <joint name="base_link_surface_joint" type="fixed">
@@ -372,49 +380,29 @@
   </joint>
   <link name="surface"/>
-  <transmission name="left_wheel_trans">
-    <type>transmission_interface/SimpleTransmission</type>
-    <joint name="left_wheel_joint">
-      <hardwareInterface>hardware_interface/VelocityJointInterface</hardwareInterface>
-    </joint>
-    <actuator name="left_wheel_motor">
-      <hardwareInterface>hardware_interface/VelocityJointInterface</hardwareInterface>
-      <mechanicalReduction>1</mechanicalReduction>
-    </actuator>
-  </transmission>
-  <transmission name="right_wheel_trans">
-    <type>transmission_interface/SimpleTransmission</type>
-    <joint name="right_wheel_joint">
-      <hardwareInterface>hardware_interface/VelocityJointInterface</hardwareInterface>
-    </joint>
-    <actuator name="right_wheel_motor">
-      <hardwareInterface>hardware_interface/VelocityJointInterface</hardwareInterface>
-      <mechanicalReduction>1</mechanicalReduction>
-    </actuator>
-  </transmission>
   <gazebo reference="left_wheel_link">
-    <mu1>1.0</mu1>
-    <mu2>1.0</mu2>
+    <mu1>200.0</mu1>
+    <mu2>200.0</mu2>
     <fdir1>1 0 0</fdir1>
   </gazebo>
   <gazebo reference="right_wheel_link">
-    <mu1>1.0</mu1>
-    <mu2>1.0</mu2>
+    <mu1>200.0</mu1>
+    <mu2>200.0</mu2>
     <fdir1>1 0 0</fdir1>
   </gazebo>
   <gazebo reference="fl_caster_wheel_link">
-    <mu1>0.001</mu1>
-    <mu2>0.001</mu2>
+    <mu1>0.0</mu1>
+    <mu2>0.0</mu2>
   </gazebo>
   <gazebo reference="fr_caster_wheel_link">
-    <mu1>0.001</mu1>
-    <mu2>0.001</mu2>
+    <mu1>0.0</mu1>
+    <mu2>0.0</mu2>
   </gazebo>
   <gazebo reference="bl_caster_wheel_link">
-    <mu1>0.001</mu1>
-    <mu2>0.001</mu2>
+    <mu1>0.0</mu1>
+    <mu2>0.0</mu2>
   </gazebo>
   <gazebo reference="br_caster_wheel_link">
-    <mu1>0.001</mu1>
-    <mu2>0.001</mu2>
+    <mu1>0.0</mu1>
+    <mu2>0.0</mu2>
   </gazebo>
   <gazebo>

File: src/mir_description/urdf/sensors/sick_lidar.xacro (robot description, xacro)
@@ -74,5 +74,5 @@
           </scan>
           <range>
-            <min>0.1</min>
+            <min>0.25</min>
             <max>30.0</max>
             <resolution>0.01</resolution>

File: src/mobile_manipulator_description/urdf/mobile_manipulator.gazebo.xacro (robot description, xacro)
@@ -7,5 +7,7 @@
     <plugin filename="gz-sim-joint-state-publisher-system"
             name="gz::sim::systems::JointStatePublisher">
-      <topic>joint_states</topic>
+      <topic>/joint_states</topic>
+      <joint_name>left_wheel_joint</joint_name>
+      <joint_name>right_wheel_joint</joint_name>
       <joint_name>ur5e_shoulder_pan_joint</joint_name>
       <joint_name>ur5e_shoulder_lift_joint</joint_name>
@@ -49,9 +51,9 @@
       <max_angular_velocity>1.0</max_angular_velocity>
       <min_angular_velocity>-1.0</min_angular_velocity>
-      <topic>cmd_vel_gz</topic>
-      <odom_topic>odom_gz</odom_topic>
+      <topic>/cmd_vel_gz</topic>
+      <odom_topic>/odom_gz</odom_topic>
       <frame_id>odom</frame_id>
       <child_frame_id>base_footprint</child_frame_id>
-      <tf_topic>tf_gz</tf_topic>
+      <tf_topic>/tf_gz</tf_topic>
       <publish_odom>true</publish_odom>
       <publish_odom_tf>true</publish_odom_tf>
