Commit message: feat(gazebo): Spawn robot in Gazebo and verify controllers and transforms

File: src/mobile_manipulator_description/urdf/mobile_manipulator.gazebo.xacro (robot description, xacro)
@@ -23,3 +23,57 @@
   <gazebo reference="ur5e_wrist_2_link"><self_collide>true</self_collide></gazebo>
   <gazebo reference="ur5e_wrist_3_link"><self_collide>true</self_collide></gazebo>
+  <!-- ros2_control configuration for Gazebo Harmonic -->
+  <ros2_control name="gz_ros2_control" type="system">
+    <hardware>
+      <plugin>gz_ros2_control/GazeboSimSystem</plugin>
+    </hardware>
+    <!-- MiR250 Base Wheels -->
+    <joint name="left_wheel_joint">
+      <command_interface name="velocity" />
+      <state_interface name="position" />
+      <state_interface name="velocity" />
+    </joint>
+    <joint name="right_wheel_joint">
+      <command_interface name="velocity" />
+      <state_interface name="position" />
+      <state_interface name="velocity" />
+    </joint>
+    <!-- UR5e Arm Joints -->
+    <joint name="ur5e_shoulder_pan_joint">
+      <command_interface name="position" />
+      <state_interface name="position" />
+      <state_interface name="velocity" />
+    </joint>
+    <joint name="ur5e_shoulder_lift_joint">
+      <command_interface name="position" />
+      <state_interface name="position" />
+      <state_interface name="velocity" />
+    </joint>
+    <joint name="ur5e_elbow_joint">
+      <command_interface name="position" />
+      <state_interface name="position" />
+      <state_interface name="velocity" />
+    </joint>
+    <joint name="ur5e_wrist_1_joint">
+      <command_interface name="position" />
+      <state_interface name="position" />
+      <state_interface name="velocity" />
+    </joint>
+    <joint name="ur5e_wrist_2_joint">
+      <command_interface name="position" />
+      <state_interface name="position" />
+      <state_interface name="velocity" />
+    </joint>
+    <joint name="ur5e_wrist_3_joint">
+      <command_interface name="position" />
+      <state_interface name="position" />
+      <state_interface name="velocity" />
+    </joint>
+  </ros2_control>
+  <!-- Gazebo ros2_control plugin -->
+  <gazebo>
+    <plugin filename="gz_ros2_control-system" name="gz_ros2_control::GazeboSimROS2ControlPlugin">
+      <parameters>$(find mobile_manipulator_gazebo)/config/gazebo_controllers.yaml</parameters>
+    </plugin>
+  </gazebo>
 </robot>

Commit message: feat: add parallel jaw gripper mechanism with controller, URDF configuration, and MoveIt integration

File: src/mobile_manipulator_description/urdf/mobile_manipulator.gazebo.xacro (robot description, xacro)
@@ -16,12 +16,10 @@
       <joint_name>ur5e_wrist_2_joint</joint_name>
       <joint_name>ur5e_wrist_3_joint</joint_name>
+      <joint_name>finger_left_joint</joint_name>
+      <joint_name>finger_right_joint</joint_name>
       <joint_name>fl_caster_rotation_joint</joint_name>
-      <joint_name>fl_caster_wheel_joint</joint_name>
       <joint_name>fr_caster_rotation_joint</joint_name>
-      <joint_name>fr_caster_wheel_joint</joint_name>
       <joint_name>bl_caster_rotation_joint</joint_name>
-      <joint_name>bl_caster_wheel_joint</joint_name>
       <joint_name>br_caster_rotation_joint</joint_name>
-      <joint_name>br_caster_wheel_joint</joint_name>
     </plugin>
   </gazebo>
@@ -105,4 +103,15 @@
       <state_interface name="velocity" />
     </joint>
+    <!-- Gripper Joints -->
+    <joint name="finger_left_joint">
+      <command_interface name="position" />
+      <state_interface name="position" />
+      <state_interface name="velocity" />
+    </joint>
+    <joint name="finger_right_joint">
+      <command_interface name="position" />
+      <state_interface name="position" />
+      <state_interface name="velocity" />
+    </joint>
   </ros2_control>
   <!-- Gazebo ros2_control plugin -->

File: src/mobile_manipulator_description/urdf/mobile_manipulator.urdf.xacro (robot description, xacro)
@@ -54,3 +54,65 @@
     <origin xyz="0 0 0" rpy="0 0 0" />
   </xacro:ur_robot>
+  <!-- Simple Parallel Jaw Gripper fingers -->
+  <!-- Left Finger -->
+  <link name="finger_left">
+    <visual>
+      <origin xyz="0.0 0.0 0.03" rpy="0 0 0" />
+      <geometry>
+        <box size="0.02 0.01 0.06" />
+      </geometry>
+      <material name="grey">
+        <color rgba="0.5 0.5 0.5 1.0" />
+      </material>
+    </visual>
+    <collision>
+      <origin xyz="0.0 0.0 0.03" rpy="0 0 0" />
+      <geometry>
+        <box size="0.02 0.01 0.06" />
+      </geometry>
+    </collision>
+    <inertial>
+      <origin xyz="0.0 0.0 0.03" rpy="0 0 0" />
+      <mass value="0.1" />
+      <inertia ixx="0.00003" ixy="0.0" ixz="0.0" iyy="0.00003" iyz="0.0" izz="0.000002" />
+    </inertial>
+  </link>
+  <!-- Right Finger -->
+  <link name="finger_right">
+    <visual>
+      <origin xyz="0.0 0.0 0.03" rpy="0 0 0" />
+      <geometry>
+        <box size="0.02 0.01 0.06" />
+      </geometry>
+      <material name="grey">
+        <color rgba="0.5 0.5 0.5 1.0" />
+      </material>
+    </visual>
+    <collision>
+      <origin xyz="0.0 0.0 0.03" rpy="0 0 0" />
+      <geometry>
+        <box size="0.02 0.01 0.06" />
+      </geometry>
+    </collision>
+    <inertial>
+      <origin xyz="0.0 0.0 0.03" rpy="0 0 0" />
+      <mass value="0.1" />
+      <inertia ixx="0.00003" ixy="0.0" ixz="0.0" iyy="0.00003" iyz="0.0" izz="0.000002" />
+    </inertial>
+  </link>
+  <!-- Prismatic joints for gripper fingers -->
+  <joint name="finger_left_joint" type="prismatic">
+    <parent link="ur5e_tool0" />
+    <child link="finger_left" />
+    <origin xyz="0.0 0.01 0.0" rpy="0 0 0" />
+    <axis xyz="0 1 0" />
+    <limit lower="0.0" upper="0.04" effort="50.0" velocity="0.1" />
+  </joint>
+  <joint name="finger_right_joint" type="prismatic">
+    <parent link="ur5e_tool0" />
+    <child link="finger_right" />
+    <origin xyz="0.0 -0.01 0.0" rpy="0 0 0" />
+    <axis xyz="0 -1 0" />
+    <limit lower="0.0" upper="0.04" effort="50.0" velocity="0.1" />
+  </joint>
 </robot>
