Commit message: feat: improve mobile manipulation robustness with base placement guardrails, higher gripper friction, updated navigation parameters, and mission retreat support. PTCHING Placing bug

File: src/mobile_manipulator_description/urdf/mobile_manipulator.gazebo.xacro (robot description, xacro)
@@ -31,4 +31,19 @@
   <gazebo reference="ur5e_wrist_2_link"><self_collide>false</self_collide></gazebo>
   <gazebo reference="ur5e_wrist_3_link"><self_collide>false</self_collide></gazebo>
+  <!-- High friction on gripper fingers to prevent object slipping -->
+  <gazebo reference="finger_left">
+    <mu1>100.0</mu1>
+    <mu2>100.0</mu2>
+    <minDepth>0.001</minDepth>
+    <kp>1000000.0</kp>
+    <kd>100.0</kd>
+  </gazebo>
+  <gazebo reference="finger_right">
+    <mu1>100.0</mu1>
+    <mu2>100.0</mu2>
+    <minDepth>0.001</minDepth>
+    <kp>1000000.0</kp>
+    <kd>100.0</kd>
+  </gazebo>
   <!-- ros2_control configuration for Gazebo Harmonic -->
   <!-- Native Gazebo DiffDrive plugin (force/torque based - works with DART physics) -->

File: src/mobile_manipulator_description/urdf/mobile_manipulator.urdf.xacro (robot description, xacro)
@@ -107,5 +107,5 @@
     <origin xyz="0.0 0.01 0.0" rpy="0 0 0" />
     <axis xyz="0 1 0" />
-    <limit lower="-0.001" upper="0.04" effort="50.0" velocity="0.1" />
+    <limit lower="-0.001" upper="0.04" effort="300.0" velocity="0.1" />
   </joint>
   <joint name="finger_right_joint" type="prismatic">
@@ -114,5 +114,5 @@
     <origin xyz="0.0 -0.01 0.0" rpy="0 0 0" />
     <axis xyz="0 -1 0" />
-    <limit lower="-0.001" upper="0.04" effort="50.0" velocity="0.1" />
+    <limit lower="-0.001" upper="0.04" effort="300.0" velocity="0.1" />
   </joint>
   <!-- Wrist depth camera for visual servoing -->
