Commit message: feat: add custom UR5e joint limits and safety collision volume to mobile manipulator description

File: src/mobile_manipulator_description/urdf/mobile_manipulator.urdf.xacro (robot description, xacro)
@@ -8,5 +8,5 @@
   <xacro:arg name="ur_type" default="ur5e" />
   <xacro:arg name="tf_prefix" default="ur5e_" />
-  <xacro:arg name="joint_limit_params" default="$(find ur_description)/config/$(arg ur_type)/joint_limits.yaml" />
+  <xacro:arg name="joint_limit_params" default="$(find mobile_manipulator_description)/config/ur5e_joint_limits.yaml" />
   <xacro:arg name="kinematics_params" default="$(find ur_description)/config/$(arg ur_type)/default_kinematics.yaml" />
   <xacro:arg name="physical_params" default="$(find ur_description)/config/$(arg ur_type)/physical_parameters.yaml" />
@@ -22,4 +22,18 @@
     <parent link="surface" />
     <child link="ur5e_mount_link" />
+    <origin xyz="0.0 0.0 0.0" rpy="0.0 0.0 0.0" />
+  </joint>
+  <!-- Safety collision volume for the mobile base to prevent self-collision -->
+  <link name="safety_collision_volume">
+    <collision>
+      <origin xyz="0.0 0.0 -0.15" rpy="0.0 0.0 0.0" />
+      <geometry>
+        <cylinder radius="0.50" length="0.40" />
+      </geometry>
+    </collision>
+  </link>
+  <joint name="safety_collision_joint" type="fixed">
+    <parent link="surface" />
+    <child link="safety_collision_volume" />
     <origin xyz="0.0 0.0 0.0" rpy="0.0 0.0 0.0" />
   </joint>

Commit message: chore: update maze origin coordinates and replace base collision cylinder with box geometry

File: src/mobile_manipulator_description/urdf/mobile_manipulator.urdf.xacro (robot description, xacro)
@@ -29,5 +29,5 @@
       <origin xyz="0.0 0.0 -0.15" rpy="0.0 0.0 0.0" />
       <geometry>
-        <cylinder radius="0.50" length="0.30" />
+        <box size="0.99 0.68 0.30" />
       </geometry>
     </collision>

Commit message: fix(orchestrator): resolve gripper prismatic limits and stowed arm self-collisions, ensuring successful end-to-end mission run and all test passing

File: src/mobile_manipulator_description/urdf/mobile_manipulator.urdf.xacro (robot description, xacro)
@@ -107,5 +107,5 @@
     <origin xyz="0.0 0.01 0.0" rpy="0 0 0" />
     <axis xyz="0 1 0" />
-    <limit lower="0.0" upper="0.04" effort="50.0" velocity="0.1" />
+    <limit lower="-0.001" upper="0.04" effort="50.0" velocity="0.1" />
   </joint>
   <joint name="finger_right_joint" type="prismatic">
@@ -114,5 +114,5 @@
     <origin xyz="0.0 -0.01 0.0" rpy="0 0 0" />
     <axis xyz="0 -1 0" />
-    <limit lower="0.0" upper="0.04" effort="50.0" velocity="0.1" />
+    <limit lower="-0.001" upper="0.04" effort="50.0" velocity="0.1" />
   </joint>
 </robot>
