Commit message: feat: update gripper joint limits, add collision exclusions, and reconfigure placement zones as open-top containers with vertical retraction paths.

File: src/mobile_manipulator_description/urdf/mobile_manipulator.urdf.xacro (robot description, xacro)
@@ -107,5 +107,5 @@
     <origin xyz="0.0 0.01 0.0" rpy="0 0 0" />
     <axis xyz="0 1 0" />
-    <limit lower="-0.001" upper="0.04" effort="300.0" velocity="0.1" />
+    <limit lower="-0.001" upper="0.04" effort="300.0" velocity="0.5" />
   </joint>
   <joint name="finger_right_joint" type="prismatic">
@@ -114,5 +114,5 @@
     <origin xyz="0.0 -0.01 0.0" rpy="0 0 0" />
     <axis xyz="0 -1 0" />
-    <limit lower="-0.001" upper="0.04" effort="300.0" velocity="0.1" />
+    <limit lower="-0.001" upper="0.04" effort="300.0" velocity="0.5" />
   </joint>
   <!-- Wrist depth camera for visual servoing -->

Commit message: Finally pick works again

File: src/mobile_manipulator_description/urdf/mobile_manipulator.urdf.xacro (robot description, xacro)
@@ -60,5 +60,5 @@
       <origin xyz="0.0 0.0 0.03" rpy="0 0 0" />
       <geometry>
-        <box size="0.02 0.01 0.06" />
+        <box size="0.02 0.01 0.12" />
       </geometry>
       <material name="grey">
@@ -69,5 +69,5 @@
       <origin xyz="0.0 0.0 0.03" rpy="0 0 0" />
       <geometry>
-        <box size="0.02 0.01 0.06" />
+        <box size="0.02 0.01 0.12" />
       </geometry>
     </collision>
@@ -83,5 +83,5 @@
       <origin xyz="0.0 0.0 0.03" rpy="0 0 0" />
       <geometry>
-        <box size="0.02 0.01 0.06" />
+        <box size="0.02 0.01 0.12" />
       </geometry>
       <material name="grey">
@@ -92,5 +92,5 @@
       <origin xyz="0.0 0.0 0.03" rpy="0 0 0" />
       <geometry>
-        <box size="0.02 0.01 0.06" />
+        <box size="0.02 0.01 0.12" />
       </geometry>
     </collision>

Commit message: pick is working perfect

File: src/mobile_manipulator_description/urdf/mobile_manipulator.urdf.xacro (robot description, xacro)
@@ -107,5 +107,8 @@
     <origin xyz="0.0 0.01 0.0" rpy="0 0 0" />
     <axis xyz="0 1 0" />
-    <limit lower="-0.001" upper="0.04" effort="300.0" velocity="0.5" />
+    <!-- limit: lower=-0.001 (fully open, inward) upper=0.041 (closed+1mm buffer)
+         The extra 1mm buffer prevents MoveIt CheckStartStateBounds from rejecting
+         the gripper-open plan when joint state feedback lands exactly at 0.04. -->
+    <limit lower="-0.001" upper="0.041" effort="300.0" velocity="0.5" />
   </joint>
   <joint name="finger_right_joint" type="prismatic">
@@ -114,5 +117,6 @@
     <origin xyz="0.0 -0.01 0.0" rpy="0 0 0" />
     <axis xyz="0 -1 0" />
-    <limit lower="-0.001" upper="0.04" effort="300.0" velocity="0.5" />
+    <!-- Same buffer as finger_left_joint -->
+    <limit lower="-0.001" upper="0.041" effort="300.0" velocity="0.5" />
   </joint>
   <!-- Wrist depth camera for visual servoing -->

Commit message: feat: expand gripper joint position limits to prevent MoveIt planning failures and add a joint state monitor script

File: src/mobile_manipulator_description/urdf/mobile_manipulator.urdf.xacro (robot description, xacro)
@@ -107,8 +107,8 @@
     <origin xyz="0.0 0.01 0.0" rpy="0 0 0" />
     <axis xyz="0 1 0" />
-    <!-- limit: lower=-0.001 (fully open, inward) upper=0.041 (closed+1mm buffer)
-         The extra 1mm buffer prevents MoveIt CheckStartStateBounds from rejecting
-         the gripper-open plan when joint state feedback lands exactly at 0.04. -->
-    <limit lower="-0.001" upper="0.041" effort="300.0" velocity="0.5" />
+    <!-- limit: lower=-0.01 (closed with buffer) upper=0.06 (open with buffer)
+         The extra buffers prevent MoveIt CheckStartStateBounds from rejecting
+         the gripper plans when joint state feedback drifts due to object contact. -->
+    <limit lower="-0.01" upper="0.06" effort="300.0" velocity="0.5" />
   </joint>
   <joint name="finger_right_joint" type="prismatic">
@@ -118,5 +118,5 @@
     <axis xyz="0 -1 0" />
     <!-- Same buffer as finger_left_joint -->
-    <limit lower="-0.001" upper="0.041" effort="300.0" velocity="0.5" />
+    <limit lower="-0.01" upper="0.06" effort="300.0" velocity="0.5" />
   </joint>
   <!-- Wrist depth camera for visual servoing -->
